File: TPS40305_supply.kicad_sch (KiCad schematic)
At the start: 31 parts, among them J1 Conn_01x01, J2 Conn_01x01, J3 Conn_01x01, J4 Conn_01x01, Q1 CSD16340Q3, Q2 CSD17311Q5, U1 TPS40305

Commit message: readme update after building R1 boards
Parts:
- U1: DK 296-25487-1-ND -> 296-37445-1-ND; PARTNO TPS40305DRCT -> TPS40305DRCR
Changed lines of the file:
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@@
       (effects (font (size 1.27 1.27)) hide)
     )
-    (property "DK" "296-25487-1-ND" (id 4) (at 142.24 100.33 0)
+    (property "DK" "296-37445-1-ND" (id 4) (at 142.24 100.33 0)
       (effects (font (size 1.27 1.27)) hide)
     )
-    (property "PARTNO" "TPS40305DRCT" (id 5) (at 142.24 100.33 0)
+    (property "PARTNO" "TPS40305DRCR" (id 5) (at 142.24 100.33 0)
       (effects (font (size 1.27 1.27)) hide)
     )
